File: cad/BlackIce_V.brd (EAGLE design)
At the start: 64 x 53 mm, 62 parts, among them IC1 REG1117, IC2 STM32F103C6T7A, IC3 ICE40UP5K, IC4 SPX3819M5_1_2, IC5 AT25SDF041A, IC6 AT25SDF041A, X1 HC49UP

Commit message: Cleaned up the schematic a little and soretyed the Pmod signals (shared with Cam data)
Connections:
- net +3V3: now also PMOD.1, PMOD.2
- net CD0: now also PMOD.10
- net CD1: now also PMOD.12
- net CD2: now also PMOD.11
- net CD3: now also PMOD.9
- net CD4: now also PMOD.7
- net CD5: now also PMOD.8
- net CD6: now also PMOD.5
- net CD7: now also PMOD.6
- net GND: now also PMOD.3, PMOD.4
